Commit message: vito for sensor fusion with gamma force torque sensor

File: vito_description/model/cylinder.urdf.xacro (robot description, xacro)
@@ -1,13 +1,21 @@
 <?xml version="1.0"?>
 <robot xmlns:xacro="http://www.ros.org/wiki/xacro" name="cylinder">
+	<xacro:macro name="cylinder_inertia_def" params="radius length mass">
+	<inertia ixx="${mass * (3 * radius * radius + length * length) / 12}"
+			 iyy="${mass * radius* radius / 2}"
+			 izz="${mass * (3 * radius * radius + length * length) / 12}"
+			 ixy="0" iyz="0" ixz="0"/>
+	</xacro:macro>
 	<link name="cylinder">
 		<inertial>
-			<mass value="0.3"/>
 			<!-- cylindrical shell : Izz=m*r^2; Ixx=Iyy=1/12*m*(6*r^2+h^2) -->
 			<!-- solid cylinder : Izz=(m*r^2)/2; Ixx=Iyy=1/12*m*(3*r^2+h^2) -->
-			<inertia  ixx="0.002385" ixy="0.00"  ixz="0.00" iyy="0.002385" iyz="0.00" izz="0.00027" />
+			<!-- <inertia  ixx="0.002385" ixy="0.00"  ixz="0.00" iyy="0.002385" iyz="0.00" izz="0.00027" /> -->
+				<mass value="0.3"/>
+				<origin xyz="0 0 0.15"  />
+				<xacro:cylinder_inertia_def radius="0.03" length="0.3" mass="0.3" />
 		</inertial>
 		<visual>
-			<origin xyz="0 0 0" rpy="0 0 0"/>
+			<origin xyz="0 0 0.15" rpy="0 0 0"/>
 			<geometry>
 				<cylinder length="0.3" radius="0.03"/>
@@ -15,5 +23,5 @@
 		</visual>
 		<collision>
-			<origin xyz="0 0 0" rpy="0 0 0"/>
+			<origin xyz="0 0 0.15" rpy="0 0 0"/>
 			<geometry>
 				<cylinder length="0.3" radius="0.03"/>
@@ -21,11 +29,11 @@
 		</collision>
 	</link>
-	<!-- <gazebo reference="cylinder"> -->
-		<!--selfCollide>true</selfCollide-->
-		<!-- <gravity>false</gravity> -->
-		<!-- <mu1>1.0</mu1> -->
-		<!-- <mu2>1.0</mu2> -->
-		<!-- <kp>10000000.0</kp> -->
-		<!-- <kd>1.0</kd> -->
-	<!-- </gazebo> -->
+	<gazebo reference="cylinder">
+		<!-- <selfCollide>true</selfCollide -->
+	     <gravity>true</gravity>
+		<mu1>0.6</mu1>
+	     <mu2>0.6</mu2>
+		<kp>10000.0</kp>
+	  <kd>100.0</kd>
+	 </gazebo>
 </robot>

File: vito_description/robot/vito.urdf_conflict-20151217-131330.xacro (robot description, xacro)
@@ -42,8 +42,8 @@
   </xacro:ft_sensor>
   <!-- LEFT SOFTHAND -->
-    <xacro:soft_hand parent="left_measure" name="left_hand" left="true" withAdaptiveTransmission="true" useMimicTag="$(arg use_mimic_tag)">
+   <xacro:soft_hand parent="left_gamma_measure" name="left_hand" left="true" withAdaptiveTransmission="true" useMimicTag="$(arg use_mimic_tag)">
     <origin xyz="0 0 0" rpy="0 0 0"/>
   </xacro:soft_hand>
-<!--   <xacro:soft_hand parent="left_measure" name="left_hand" left="true" withAdaptiveTransmission="true" useMimicTag="true">
+<!--   <xacro:soft_hand parent="left_gamma_measure" name="left_hand" left="true" withAdaptiveTransmission="true" useMimicTag="true">
     <origin xyz="0 0 0" rpy="0 0 0"/>
   </xacro:soft_hand> -->
@@ -57,10 +57,10 @@
   </xacro:ft_sensor>
   <!-- RIGHT SOFTHAND -->
-    <xacro:soft_hand parent="right_measure" name="right_hand" left="false" withAdaptiveTransmission="true" useMimicTag="$(arg use_mimic_tag)">
+   <xacro:soft_hand parent="right_gamma_measure" name="right_hand" left="false" withAdaptiveTransmission="true" useMimicTag="$(arg use_mimic_tag)">
     <origin xyz="0 0 0" rpy="0 0 0"/>
   </xacro:soft_hand>
-<!--   <xacro:soft_hand parent="right_measure" name="right_hand" left="false" withAdaptiveTransmission="true" useMimicTag="true">
+<!--   <xacro:soft_hand parent="right_gamma_measure" name="right_hand" left="false" withAdaptiveTransmission="true" useMimicTag="true">
     <origin xyz="0 0 0" rpy="0 0 0"/>
-  </xacro:soft_hand>  -->
+  </xacro:soft_hand> -->
   <!-- HEAD -->
   <xacro:kit_head name="head" parent="vito_anchor">

Commit message: vito for sensor fusion with gazebo gripper

File: vito_description/model/cylinder.urdf.xacro (robot description, xacro)
@@ -3,6 +3,6 @@
 	<xacro:macro name="cylinder_inertia_def" params="radius length mass">
 	<inertia ixx="${mass * (3 * radius * radius + length * length) / 12}"
-			 iyy="${mass * radius* radius / 2}"
-			 izz="${mass * (3 * radius * radius + length * length) / 12}"
+			 iyy="${mass * (3 * radius * radius + length * length) / 12}"
+			 izz="${mass * radius* radius / 2}"
 			 ixy="0" iyz="0" ixz="0"/>
 	</xacro:macro>
@@ -12,28 +12,33 @@
 			<!-- solid cylinder : Izz=(m*r^2)/2; Ixx=Iyy=1/12*m*(3*r^2+h^2) -->
 			<!-- <inertia  ixx="0.002385" ixy="0.00"  ixz="0.00" iyy="0.002385" iyz="0.00" izz="0.00027" /> -->
-				<mass value="0.3"/>
-				<origin xyz="0 0 0.15"  />
-				<xacro:cylinder_inertia_def radius="0.03" length="0.3" mass="0.3" />
+				<mass value="1.0"/>
+				<origin xyz="0 0 0.0075"/>
+				<xacro:cylinder_inertia_def radius="0.035" length="0.015" mass="1.0" />
 		</inertial>
 		<visual>
-			<origin xyz="0 0 0.15" rpy="0 0 0"/>
+			<origin xyz="0 0 0.0075" rpy="0 0 0"/>
 			<geometry>
-				<cylinder length="0.3" radius="0.03"/>
+				<cylinder length="0.015" radius="0.035"/>
 			</geometry>
 		</visual>
 		<collision>
-			<origin xyz="0 0 0.15" rpy="0 0 0"/>
+			<origin xyz="0 0 0.0075" rpy="0 0 0"/>
 			<geometry>
-				<cylinder length="0.3" radius="0.03"/>
+				<cylinder length="0.015" radius="0.035"/>
 			</geometry>
 		</collision>
 	</link>
 	<gazebo reference="cylinder">
-		<!-- <selfCollide>true</selfCollide -->
+		  <selfCollide>true</selfCollide>
+		 <maxContacts>100</maxContacts>
+	     <!-- <provideFeedback>true</provideFeedback>  -->
 	     <gravity>true</gravity>
 		<mu1>0.6</mu1>
 	     <mu2>0.6</mu2>
-		<kp>10000.0</kp>
+	        <fdir1>1 0 0</fdir1>
+         <maxVel>1.0</maxVel>
+		<kp>10000000.0</kp>
 	  <kd>100.0</kd>
+	  <minDepth>0.00</minDepth>
 	 </gazebo>
 </robot>

File: vito_description/robot/vito.urdf.xacro (robot description, xacro)
@@ -10,5 +10,11 @@
   <xacro:include filename="$(find kit_head_description)/model/kit_head.urdf.xacro"/>
   <xacro:include filename="$(find force_torque_sensor)/model/ft_sensor_gamma.urdf.xacro"/>
-  <link name="vito_anchor" />
+ <link name="vito_anchor" />
+<!--   <link name="world" /> -->
+<!--  <joint name="world_joint" type="fixed">
+    <origin xyz="0.0 0.0 -0.1" rpy="0 0 0"/>
+      <parent link="world"/>
+      <child link="vito_anchor"/>
+   </joint> -->
   <!-- BODY -->
   <xacro:model_table name="table"
@@ -43,5 +49,5 @@
   <!-- LEFT SOFTHAND -->
     <xacro:soft_hand parent="left_measure" name="left_hand" left="true" withAdaptiveTransmission="true" useMimicTag="$(arg use_mimic_tag)">
-    <origin xyz="0 0 0" rpy="0 0 0"/>
+    <origin xyz="0 0 0.0025" rpy="0 0 0"/>
   </xacro:soft_hand>
 <!--   <xacro:soft_hand parent="left_measure" name="left_hand" left="true" withAdaptiveTransmission="true" useMimicTag="true">
@@ -58,5 +64,5 @@
   <!-- RIGHT SOFTHAND -->
     <xacro:soft_hand parent="right_measure" name="right_hand" left="false" withAdaptiveTransmission="true" useMimicTag="$(arg use_mimic_tag)">
-    <origin xyz="0 0 0" rpy="0 0 0"/>
+    <origin xyz="0 0 0.0025" rpy="0 0 0"/>
   </xacro:soft_hand>
 <!--   <xacro:soft_hand parent="right_measure" name="right_hand" left="false" withAdaptiveTransmission="true" useMimicTag="true">
