Commit message: VITO for sensor fusion and grasp estimation (second commit) end effector in hand _palm_dummy_link controller problem to solve

File: vito_description/robot/vito.urdf.xacro (robot description, xacro)
@@ -40,4 +40,7 @@
     <origin xyz="0 0 0" rpy="0 0 0"/>
   </xacro:soft_hand>
+<!--   <xacro:soft_hand parent="left_arm_7_link" name="left_hand" left="true" withAdaptiveTransmission="true" useMimicTag="true">
+    <origin xyz="0 0 0" rpy="0 0 0"/>
+  </xacro:soft_hand> -->
   <!-- RIGHT ARM -->
   <xacro:kuka_lwr name="right_arm" parent="vito_anchor">
@@ -48,4 +51,8 @@
     <origin xyz="0 0 0" rpy="0 0 0"/>
   </xacro:soft_hand>
+<!--
+  <xacro:soft_hand parent="right_arm_7_link" name="right_hand" left="false" withAdaptiveTransmission="true" useMimicTag="true">
+    <origin xyz="0 0 0" rpy="0 0 0"/>
+  </xacro:soft_hand> -->
   <!-- HEAD -->
   <xacro:kit_head name="head" parent="vito_anchor">

Commit message: vito robot with F/T sensor on arms

File: vito_description/robot/vito.urdf.xacro (robot description, xacro)
@@ -9,4 +9,5 @@
   <xacro:include filename="$(find soft_hand_description)/model/soft_hand.urdf.xacro"/>
   <xacro:include filename="$(find kit_head_description)/model/kit_head.urdf.xacro"/>
+  <xacro:include filename="$(find force_torque_sensor)/model/ft_sensor.urdf.xacro"/>
   <link name="vito_anchor" />
   <!-- BODY -->
@@ -36,9 +37,13 @@
     <origin xyz="-0.165 -0.1085854 0.390" rpy="1.5707963267948966 0.5235987010713441 -0.5235990737060282"/>
   </xacro:kuka_lwr>
+    <!-- LEFT F/T Sensor -->
+    <xacro:ft_sensor parent="left_arm_7_link" name="left" type="gamma">
+    <origin xyz="0 0 0" rpy="0 0 0"/>
+  </xacro:ft_sensor>
   <!-- LEFT SOFTHAND -->
-  <xacro:soft_hand parent="left_arm_7_link" name="left_hand" left="true" withAdaptiveTransmission="true" useMimicTag="$(arg use_mimic_tag)">
+   <xacro:soft_hand parent="left_gamma_measure" name="left_hand" left="true" withAdaptiveTransmission="true" useMimicTag="$(arg use_mimic_tag)">
     <origin xyz="0 0 0" rpy="0 0 0"/>
   </xacro:soft_hand>
-<!--   <xacro:soft_hand parent="left_arm_7_link" name="left_hand" left="true" withAdaptiveTransmission="true" useMimicTag="true">
+<!--   <xacro:soft_hand parent="left_gamma_measure" name="left_hand" left="true" withAdaptiveTransmission="true" useMimicTag="true">
     <origin xyz="0 0 0" rpy="0 0 0"/>
   </xacro:soft_hand> -->
@@ -47,10 +52,13 @@
     <origin xyz="-0.165 0.10858 0.390" rpy="-1.5707963267948966 0.5235987010713441 0.5235990737060282"/>
   </xacro:kuka_lwr>
+  <!-- RIGHT F/T Sensor -->
+    <xacro:ft_sensor parent="right_arm_7_link" name="right" type="gamma">
+    <origin xyz="0 0 0" rpy="0 0 0"/>
+  </xacro:ft_sensor>
   <!-- RIGHT SOFTHAND -->
-  <xacro:soft_hand parent="right_arm_7_link" name="right_hand" left="false" withAdaptiveTransmission="true" useMimicTag="$(arg use_mimic_tag)">
+   <xacro:soft_hand parent="right_gamma_measure" name="right_hand" left="false" withAdaptiveTransmission="true" useMimicTag="$(arg use_mimic_tag)">
     <origin xyz="0 0 0" rpy="0 0 0"/>
   </xacro:soft_hand>
-<!--
-  <xacro:soft_hand parent="right_arm_7_link" name="right_hand" left="false" withAdaptiveTransmission="true" useMimicTag="true">
+<!--   <xacro:soft_hand parent="right_gamma_measure" name="right_hand" left="false" withAdaptiveTransmission="true" useMimicTag="true">
     <origin xyz="0 0 0" rpy="0 0 0"/>
   </xacro:soft_hand> -->

Commit message: final version of vito for sensor fusion

File: vito_description/robot/vito.urdf.xacro (robot description, xacro)
@@ -10,11 +10,11 @@
   <xacro:include filename="$(find kit_head_description)/model/kit_head.urdf.xacro"/>
   <xacro:include filename="$(find force_torque_sensor)/model/ft_sensor_gamma.urdf.xacro"/>
- <link name="vito_anchor" />
-<!--   <link name="world" /> -->
-<!--  <joint name="world_joint" type="fixed">
-    <origin xyz="0.0 0.0 -0.1" rpy="0 0 0"/>
+<!--   <link name="world" />
+  <joint name="world_joint" type="fixed">
+    <origin xyz="0.0 0.0 -0.05" rpy="0 0 0"/>
       <parent link="world"/>
       <child link="vito_anchor"/>
    </joint> -->
+   <link name="vito_anchor" />
   <!-- BODY -->
   <xacro:model_table name="table"

Commit message: final version of vito for sensor fusion

File: vito_description/robot/vito.urdf.xacro (robot description, xacro)
@@ -45,9 +45,9 @@
     <!-- LEFT F/T Sensor -->
     <xacro:ft_sensor parent="left_arm_7_link" name="left" type="gamma">
-    <origin xyz="0 0 0" rpy="0 0 0"/>
+    <origin xyz="0 0 0.014" rpy="0 0 0"/>
   </xacro:ft_sensor>
   <!-- LEFT SOFTHAND -->
     <xacro:soft_hand parent="left_measure" name="left_hand" left="true" withAdaptiveTransmission="true" useMimicTag="$(arg use_mimic_tag)">
-    <origin xyz="0 0 0.0025" rpy="0 0 0"/>
+    <origin xyz="0 0 0.026" rpy="0 0 0"/>
   </xacro:soft_hand>
 <!--   <xacro:soft_hand parent="left_measure" name="left_hand" left="true" withAdaptiveTransmission="true" useMimicTag="true">
@@ -59,10 +59,10 @@
   </xacro:kuka_lwr>
   <!-- RIGHT F/T Sensor -->
-    <xacro:ft_sensor parent="right_arm_7_link" name="right" type="gamma">
+<!--    <xacro:ft_sensor parent="right_arm_7_link" name="right" type="gamma">
     <origin xyz="0 0 0" rpy="0 0 0"/>
-  </xacro:ft_sensor>
+  </xacro:ft_sensor>-->
   <!-- RIGHT SOFTHAND -->
-    <xacro:soft_hand parent="right_measure" name="right_hand" left="false" withAdaptiveTransmission="true" useMimicTag="$(arg use_mimic_tag)">
-    <origin xyz="0 0 0.0025" rpy="0 0 0"/>
+    <xacro:soft_hand parent="right_arm_7_link" name="right_hand" left="false" withAdaptiveTransmission="true" useMimicTag="$(arg use_mimic_tag)">
+    <origin xyz="0 0 0.026" rpy="0 0 0"/>
   </xacro:soft_hand>
 <!--   <xacro:soft_hand parent="right_measure" name="right_hand" left="false" withAdaptiveTransmission="true" useMimicTag="true">

Commit message: workin version with real robot without submodules

File: vito_description/robot/vito.urdf.xacro (robot description, xacro)
@@ -45,5 +45,5 @@
     <!-- LEFT F/T Sensor -->
     <xacro:ft_sensor parent="left_arm_7_link" name="left" type="gamma">
-    <origin xyz="0 0 0.014" rpy="0 0 0"/>
+    <origin xyz="0 0 0.031" rpy="0 0 0"/>
   </xacro:ft_sensor>
   <!-- LEFT SOFTHAND -->
